Commit message: feat: add Gazebo drive lidar and camera sensors

File: ros2_ws/src/robot_description/urdf/robot.urdf.xacro (robot description, xacro)
@@ -26,5 +26,5 @@
     </link>
     <joint name="${name}_joint" type="continuous">
-      <parent link="base_link"/><child link="${name}"/><origin xyz="${x} ${y} 0.075" rpy="0 0 0"/><axis xyz="0 1 0"/>
+      <parent link="base_link"/><child link="${name}"/><origin xyz="${x} ${y} 0.075"/><axis xyz="0 1 0"/>
     </joint>
   </xacro:macro>
@@ -46,8 +46,52 @@
   <joint name="lidar_joint" type="fixed"><parent link="base_link"/><child link="lidar_link"/><origin xyz="0 0 0.18"/></joint>
   <link name="camera_link">
-    <visual><geometry><box size="0.08 0.06 0.05"/></geometry><material name="white"/></visual>
+    <visual><geometry><box size="0.08 0.06 0.05"/></geometry><material name="white"/></material></visual>
     <collision><geometry><box size="0.08 0.06 0.05"/></geometry></collision>
     <inertial><mass value="0.1"/><inertia ixx="0.0001" ixy="0" ixz="0" iyy="0.0001" iyz="0" izz="0.0001"/></inertial>
   </link>
-  <joint name="camera_joint" type="fixed"><parent link="base_link"/><child link="camera_link"/><origin xyz="0.20 0 0.22" rpy="0 0 0"/></joint>
+  <joint name="camera_joint" type="fixed"><parent link="base_link"/><child link="camera_link"/><origin xyz="0.20 0 0.22"/></joint>
+  <!-- Gazebo Sim / Harmonic systems -->
+  <gazebo>
+    <plugin filename="gz-sim-diff-drive-system" name="gz::sim::systems::DiffDrive">
+      <left_joint>left_wheel_joint</left_joint>
+      <right_joint>right_wheel_joint</right_joint>
+      <wheel_separation>0.40</wheel_separation>
+      <wheel_radius>${wheel_radius}</wheel_radius>
+      <topic>/cmd_vel</topic>
+      <odom_topic>/odom</odom_topic>
+      <tf_topic>/tf</tf_topic>
+      <frame_id>odom</frame_id>
+      <child_frame_id>base_footprint</child_frame_id>
+      <odom_publish_frequency>30</odom_publish_frequency>
+    </plugin>
+  </gazebo>
+  <gazebo reference="lidar_link">
+    <sensor name="lidar" type="gpu_lidar">
+      <topic>/scan</topic>
+      <update_rate>10</update_rate>
+      <always_on>true</always_on>
+      <visualize>true</visualize>
+      <gz_frame_id>lidar_link</gz_frame_id>
+      <ray>
+        <scan>
+          <horizontal><samples>360</samples><resolution>1</resolution><min_angle>-3.14159</min_angle><max_angle>3.14159</max_angle></horizontal>
+        </scan>
+        <range><min>0.12</min><max>10.0</max><resolution>0.01</resolution></range>
+      </ray>
+    </sensor>
+  </gazebo>
+  <gazebo reference="camera_link">
+    <sensor name="camera" type="camera">
+      <topic>/camera/image_raw</topic>
+      <update_rate>15</update_rate>
+      <always_on>true</always_on>
+      <visualize>true</visualize>
+      <gz_frame_id>camera_link</gz_frame_id>
+      <camera>
+        <horizontal_fov>1.047</horizontal_fov>
+        <image><width>640</width><height>480</height><format>R8G8B8</format></image>
+        <clip><near>0.05</near><far>20</far></clip>
+      </camera>
+    </sensor>
+  </gazebo>
 </robot>

Commit message: fix: correct camera material XML

File: ros2_ws/src/robot_description/urdf/robot.urdf.xacro (robot description, xacro)
@@ -16,7 +16,5 @@
     <inertial><origin xyz="0 0 0.08"/><mass value="5.0"/><inertia ixx="0.08" ixy="0" ixz="0" iyy="0.12" iyz="0" izz="0.15"/></inertial>
   </link>
-  <joint name="base_footprint_joint" type="fixed">
-    <parent link="base_footprint"/><child link="base_link"/><origin xyz="0 0 0"/>
-  </joint>
+  <joint name="base_footprint_joint" type="fixed"><parent link="base_footprint"/><child link="base_link"/><origin xyz="0 0 0"/></joint>
   <xacro:macro name="wheel" params="name x y">
     <link name="${name}">
@@ -25,7 +23,5 @@
       <inertial><mass value="0.4"/><inertia ixx="0.0015" ixy="0" ixz="0" iyy="0.0015" iyz="0" izz="0.0015"/></inertial>
     </link>
-    <joint name="${name}_joint" type="continuous">
-      <parent link="base_link"/><child link="${name}"/><origin xyz="${x} ${y} 0.075"/><axis xyz="0 1 0"/>
-    </joint>
+    <joint name="${name}_joint" type="continuous"><parent link="base_link"/><child link="${name}"/><origin xyz="${x} ${y} 0.075"/><axis xyz="0 1 0"/></joint>
   </xacro:macro>
   <xacro:wheel name="left_wheel" x="0" y="${wheel_y}"/>
@@ -36,7 +32,5 @@
     <inertial><mass value="0.2"/><inertia ixx="0.0001" ixy="0" ixz="0" iyy="0.0001" iyz="0" izz="0.0001"/></inertial>
   </link>
-  <joint name="caster_joint" type="fixed">
-    <parent link="base_link"/><child link="caster_link"/><origin xyz="-0.16 0 0.045"/>
-  </joint>
+  <joint name="caster_joint" type="fixed"><parent link="base_link"/><child link="caster_link"/><origin xyz="-0.16 0 0.045"/></joint>
   <link name="lidar_link">
     <visual><geometry><cylinder radius="0.055" length="0.04"/></geometry><material name="white"/></visual>
@@ -46,51 +40,27 @@
   <joint name="lidar_joint" type="fixed"><parent link="base_link"/><child link="lidar_link"/><origin xyz="0 0 0.18"/></joint>
   <link name="camera_link">
-    <visual><geometry><box size="0.08 0.06 0.05"/></geometry><material name="white"/></material></visual>
+    <visual><geometry><box size="0.08 0.06 0.05"/></geometry><material name="white"/></visual>
     <collision><geometry><box size="0.08 0.06 0.05"/></geometry></collision>
     <inertial><mass value="0.1"/><inertia ixx="0.0001" ixy="0" ixz="0" iyy="0.0001" iyz="0" izz="0.0001"/></inertial>
   </link>
   <joint name="camera_joint" type="fixed"><parent link="base_link"/><child link="camera_link"/><origin xyz="0.20 0 0.22"/></joint>
-  <!-- Gazebo Sim / Harmonic systems -->
   <gazebo>
     <plugin filename="gz-sim-diff-drive-system" name="gz::sim::systems::DiffDrive">
-      <left_joint>left_wheel_joint</left_joint>
-      <right_joint>right_wheel_joint</right_joint>
-      <wheel_separation>0.40</wheel_separation>
-      <wheel_radius>${wheel_radius}</wheel_radius>
-      <topic>/cmd_vel</topic>
-      <odom_topic>/odom</odom_topic>
-      <tf_topic>/tf</tf_topic>
-      <frame_id>odom</frame_id>
-      <child_frame_id>base_footprint</child_frame_id>
-      <odom_publish_frequency>30</odom_publish_frequency>
+      <left_joint>left_wheel_joint</left_joint><right_joint>right_wheel_joint</right_joint>
+      <wheel_separation>0.40</wheel_separation><wheel_radius>${wheel_radius}</wheel_radius>
+      <topic>/cmd_vel</topic><odom_topic>/odom</odom_topic><tf_topic>/tf</tf_topic>
+      <frame_id>odom</frame_id><child_frame_id>base_footprint</child_frame_id><odom_publish_frequency>30</odom_publish_frequency>
     </plugin>
   </gazebo>
   <gazebo reference="lidar_link">
     <sensor name="lidar" type="gpu_lidar">
-      <topic>/scan</topic>
-      <update_rate>10</update_rate>
-      <always_on>true</always_on>
-      <visualize>true</visualize>
-      <gz_frame_id>lidar_link</gz_frame_id>
-      <ray>
-        <scan>
-          <horizontal><samples>360</samples><resolution>1</resolution><min_angle>-3.14159</min_angle><max_angle>3.14159</max_angle></horizontal>
-        </scan>
-        <range><min>0.12</min><max>10.0</max><resolution>0.01</resolution></range>
-      </ray>
+      <topic>/scan</topic><update_rate>10</update_rate><always_on>true</always_on><visualize>true</visualize><gz_frame_id>lidar_link</gz_frame_id>
+      <ray><scan><horizontal><samples>360</samples><resolution>1</resolution><min_angle>-3.14159</min_angle><max_angle>3.14159</max_angle></horizontal></scan><range><min>0.12</min><max>10.0</max><resolution>0.01</resolution></range></ray>
     </sensor>
   </gazebo>
   <gazebo reference="camera_link">
     <sensor name="camera" type="camera">
-      <topic>/camera/image_raw</topic>
-      <update_rate>15</update_rate>
-      <always_on>true</always_on>
-      <visualize>true</visualize>
-      <gz_frame_id>camera_link</gz_frame_id>
-      <camera>
-        <horizontal_fov>1.047</horizontal_fov>
-        <image><width>640</width><height>480</height><format>R8G8B8</format></image>
-        <clip><near>0.05</near><far>20</far></clip>
-      </camera>
+      <topic>/camera/image_raw</topic><update_rate>15</update_rate><always_on>true</always_on><visualize>true</visualize><gz_frame_id>camera_link</gz_frame_id>
+      <camera><horizontal_fov>1.047</horizontal_fov><image><width>640</width><height>480</height><format>R8G8B8</format></image><clip><near>0.05</near><far>20</far></clip></camera>
     </sensor>
   </gazebo>
